File: ES100-MOD Clock.kicad_pcb (KiCad board)
At the start: 2 copper layers, 25.4 x 28.6 mm, 7 parts, among them J1 ANT1, J2 ANT2, J99 mikrobus-add-on, U1 ES100-MOD-v1.1

Commit message: Add files via upload
Parts:
- J1, J2: footprint TerminalBlock_TE-Connectivity:TerminalBlock_TE_282834-2_1x02_P2.54mm_Horizontal -> footprints:TerminalBlock_TE_282834-2_1x02_P2.54mm_Horizontal
- J99: footprint ml-symbols:mikrobus-small -> footprints:mikrobus-small
- REF**: footprint ml-symbols:3v3-LOGO -> footprints:3v3-LOGO
- REF**: footprint ml-symbols:mikrobus-logo-small -> footprints:mikrobus-logo-small
- REF**: footprint Symbol:OSHW-Logo2_7.3x6mm_SilkScreen -> footprints:OSHW-Logo2_7.3x6mm_SilkScreen
- U1: footprint ml-symbols:ES100-MOD -> footprints:ES100-MOD
Changed lines of the file:
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@@
   (net 18 "/AN1+")
   (net 19 "/AN1-")
-  (footprint "ml-symbols:3v3-LOGO" (layer "F.Cu")
+  (footprint "footprints:3v3-LOGO" (layer "F.Cu")
     (at 97.286 49.74258)
     (descr "3.3V Graphical Logo")
@@
     (fp_arc (start 0.3175 0.365) (mid 0 3.311241) (end -0.3175 0.365) (layer "F.SilkS") (width 0.2032))
   )
-  (footprint "ml-symbols:mikrobus-small" (layer "F.Cu")
+  (footprint "footprints:mikrobus-small" (layer "F.Cu")
     (at 91.554 48.564)
     (property "Sheetfile" "ES100-MOD Clock.kicad_sch")
@@
       (net 9 "GND") (pinfunction "GND") (pintype "power_in"))
   )
-  (footprint "TerminalBlock_TE-Connectivity:TerminalBlock_TE_282834-2_1x02_P2.54mm_Horizontal" (layer "F.Cu")
+  (footprint "footprints:TerminalBlock_TE_282834-2_1x02_P2.54mm_Horizontal" (layer "F.Cu")
     (at 110.824 52.039 180)
     (descr "Terminal Block TE 282834-2, 2 pins, pitch 2.54mm, size 5.54x6.5mm^2, drill diamater 1.1mm, pad diameter 2.1mm, see http://www.te.com/commerce/DocumentDelivery/DDEController?Action=showdoc&DocId=Customer+Drawing%7F282834%7FC1%7Fpdf%7FEnglish%7FENG_CD_282834_C1.pdf, script-generated using https://github.com/pointhi/kicad-footprint-generator/scripts/TerminalBlock_TE-Connectivity")
@@
     )
   )
-  (footprint "TerminalBlock_TE-Connectivity:TerminalBlock_TE_282834-2_1x02_P2.54mm_Horizontal" (layer "F.Cu")
+  (footprint "footprints:TerminalBlock_TE_282834-2_1x02_P2.54mm_Horizontal" (layer "F.Cu")
     (at 104.054 52.039 180)
     (descr "Terminal Block TE 282834-2, 2 pins, pitch 2.54mm, size 5.54x6.5mm^2, drill diamater 1.1mm, pad diameter 2.1mm, see http://www.te.com/commerce/DocumentDelivery/DDEController?Action=showdoc&DocId=Customer+Drawing%7F282834%7FC1%7Fpdf%7FEnglish%7FENG_CD_282834_C1.pdf, script-generated using https://github.com/pointhi/kicad-footprint-generator/scripts/TerminalBlock_TE-Connectivity")
@@
     )
   )
-  (footprint "ml-symbols:mikrobus-logo-small" (layer "F.Cu")
+  (footprint "footprints:mikrobus-logo-small" (layer "F.Cu")
     (at 93.73 50.5145)
     (descr "mikrobus graphical logo, small")
@@
     (fp_circle (center 1.27 1.4445) (end 1.524 1.4445) (layer "F.SilkS") (width 0.1524) (fill solid))
   )
-  (footprint "ml-symbols:ES100-MOD" (layer "F.Cu")
+  (footprint "footprints:ES100-MOD" (layer "F.Cu")
     (at 96.0968 70.2088 90)
     (property "Sheetfile" "ES100-MOD Clock.kicad_sch")
@@
       (net 8 "/AN2+") (pinfunction "AN2+") (pintype "passive"))
   )
-  (footprint "Symbol:OSHW-Logo2_7.3x6mm_SilkScreen" (layer "B.Cu")
+  (footprint "footprints:OSHW-Logo2_7.3x6mm_SilkScreen" (layer "B.Cu")
     (at 107.7 64.278 180)
     (descr "Open Source Hardware Symbol")
