File: ES100-MOD Clock.kicad_sch (KiCad schematic)
At the start: 4 parts, among them J1 ANT1, J2 ANT2, J99 Mikrobus Add-On Footprint, U1 ES100-MOD-v1.1

Commit message: Add files via upload
Other:
- moved on the sheet: J1, J2, J99, U1
